File: GaN-inverter_design.kicad_sch (KiCad schematic)
At the start: 34 parts, among them U1 LMG2100R026VBNR, U2 INA240A1D, U3 SN74LVC245APW, U4 LMG2100R026VBNR, U5 INA240A1D, U6 LMG2100R026VBNR, U7 INA240A1D

Commit message: updates
Parts:
- removed C1, C10, C11, C12, C13, C14, C15, C2, C3, C4, C5, C6, C7, C8, C9: C, symbol Device:C
- removed R1, R10, R11, R12, R2, R3, R4, R5, R6, R7, R8, R9: R, symbol Device:R
- removed U1, U4, U6: LMG2100R026VBNR, LMG2100:VBN0018A-MFG, symbol LMG2100:LMG2100R026VBNR
- removed U2, U5, U7: INA240A1D, Package_SO:SOIC-8_3.9x4.9mm_P1.27mm, symbol Amplifier_Current:INA240A1D
Connections:
- net power_stage2/HI: now reaches U3.14 (B5)
- net power_stage/LI: now reaches U3.17 (B2)
- net power_stage1/HI: now reaches U3.16 (B3)
- net power_stage2/LI: now reaches U3.13 (B6)
- net power_stage1/LI: now reaches U3.15 (B4)
- net power_stage/HI: now reaches U3.18 (B1)
Other:
- added sheet DC-DC buck (untitled.kicad_sch)
- added sheet housekeeping (housekeeping.kicad_sch)
- added sheet microcontroller (microcontroller.kicad_sch)
- added sheet power_stage (power_stage.kicad_sch)
- added sheet power_stage1 (power_stage.kicad_sch)
- added sheet power_stage2 (power_stage.kicad_sch)
